File: 03_power.kicad_sch (KiCad schematic)
At the start: 19 parts, among them J1 15V INPUT, U3 TPS62163DSGR, U4 TPS62162DSGR, U5 TPS62161DSGR

Commit message: Rev D schematic: ГОСТ symbols and designators in KiCad, footprints
- Three sheets regenerated by tools/dds_build.py (DDS A2, controller A3,
  power A2) with ГОСТ 2.743 symbols, ГОСТ 2.710 designators (D1.1, XW1, S2)
  and a ГОСТ 2.104 drawing sheet (lib/GOST_E3.kicad_wks).
- Connectivity identical to rev C (tools/netcompare.py with
  verification/refmap_revC_to_revD.json): 160 components, 139 nets; the 12
  single DIP switches are grouped into DIP-8 + DIP-4 packages.
- ERC: 0 errors, 0 warnings. Footprints assigned; project library lib/
  (1508PL8T LQFP-100, 1887VE7T CQFP-64 4203.64-2 preliminary, GK361-TK-02
  placeholder - not confirmed, DNP).
- Old rev C PDF replaced by output/pdf/DDS_47_51_sch.pdf.

Co-Authored-By: Claude Opus 5.5 <noreply@anthropic.com>
Claude-Session: https://claude.ai/code/session_018GorfTmWz53k1K9rRxWMAW
Parts:
- removed C1, C4, C7: 10u / 25V, symbol Local:C
- removed C2, C5, C8: 22u / 10V, symbol Local:C
- removed C3, C6, C9: 100n, symbol Local:C
- removed D1: SS34, symbol Local:D_Schottky
- removed F1: 0.5A, symbol Local:Fuse
- removed J1: 15V INPUT, symbol Local:J2
- removed L1, L2, L3: 2.2u / Isat>=1.5A, symbol Local:L
- removed R1: 47k, symbol Local:R
- removed U3: TPS62163DSGR, symbol Local:TPS6216x
- removed U4: TPS62162DSGR, symbol Local:TPS6216x
- removed U5: TPS62161DSGR, symbol Local:TPS6216x
- added C46, C49, C52: 10u, Capacitor_SMD:C_1206_3216Metric, symbol DDS:C
- added C47, C50, C53: 100n, Capacitor_SMD:C_0603_1608Metric, symbol DDS:C
- added C48, C51, C54: 22u, Capacitor_SMD:C_1206_3216Metric, symbol DDS:C
- added D5: TPS62163DSGR, Package_SON:Texas_DSG0008A_WSON-8-1EP_2x2mm_P0.5mm_EP0.9x1.6mm, symbol DDS:TPS6216x
- added D6: TPS62162DSGR, Package_SON:Texas_DSG0008A_WSON-8-1EP_2x2mm_P0.5mm_EP0.9x1.6mm, symbol DDS:TPS6216x
- added D7: TPS62161DSGR, Package_SON:Texas_DSG0008A_WSON-8-1EP_2x2mm_P0.5mm_EP0.9x1.6mm, symbol DDS:TPS6216x
- added F1: 0.5A, Fuse:Fuse_1206_3216Metric, symbol DDS:F
- added L10, L8, L9: 2.2u, Inductor_SMD:L_Changjiang_FNR4020S, symbol DDS:L
- added R78: 47k, Resistor_SMD:R_0603_1608Metric, symbol DDS:R
- added VD1: SS34, Diode_SMD:D_SMA, symbol DDS:VD_Schottky
- added X2: PLS-2, Connector_PinHeader_2.54mm:PinHeader_1x02_P2.54mm_Vertical, symbol DDS:X_2
Connections:
- net +1V8: now also C54.1, D7.6 (VOS), L10.2
- net +3V3: now also C51.1, D6.6 (VOS), L9.2
- net +5V: now also C48.1, C49.1, C50.1, C52.1, C53.1, D5.6 (VOS), D6.2 (VIN), D6.3 (EN), D7.2 (VIN), D7.3 (EN), L8.2, R78.1
- net DDS_PGOOD: now also D6.8 (PG), D7.8 (PG), R78.2
- net GND: now also C46.2, C47.2, C48.2, C49.2, C50.2, C51.2, C52.2, C53.2, C54.2, D5.1 (PGND), D5.4 (AGND), D5.5 (FB), D5.9 (EP), D6.1 (PGND), D6.4 (AGND), D6.5 (FB), D6.9 (EP), D7.1 (PGND), D7.4 (AGND), D7.5 (FB), D7.9 (EP), X2.2
- net MCU_RESETn: now also D5.8 (PG)
- net VIN_PROT: now also C46.1, C47.1, D5.2 (VIN), D5.3 (EN), VD1.1 (K)
- new net: D7.7 (SW), L10.1
- new net: D6.7 (SW), L9.1
- new net: D5.7 (SW), L8.1
- new net: F1.1, X2.1
- new net: F1.2, VD1.2 (A)
Other:
- note added: "+15 В ±5 %"
- note added: "1. Вход +15 В ±5 %; напряжение на входе D5 должно оставаться ниже 17 В."
- note added: "2. VD1 — защита от обратной полярности, F1 — от перегрузки."
- note added: "3. Ёмкости указаны эффективными при рабочем напряжении, диэлектрик X7R."
- note added: "4. Тепловые площадки D5–D7 соединить с GND; контуры SW — минимальной длины."
- note added: "5. PG D5 формирует сброс МК; PG D6, D7 — признак готовности питания DDS."
- note added: "6. Бюджет: 1,8 В <= 0,4 А (DDS); 3,3 В <= 0,2 А + генератор G1 (уточнить)."
- note added: "PG D6, D7 — монтажное И: питание DDS в норме"
- note added: "Примечания"
- note removed: "03 POWER / preliminary circuit"
- note removed: "Input +15 V +/-5%; VIN <17 V. Effective capacitance at DC bias. PG U4/U5 wired-AND. Verify oscillator current, thermal and noise performance."
- title: Power supply / +15 V input -> Синтезатор частоты 47–51 МГц

Commit message: Rev E: domestic regulators and logic (1393ЕУ014 + LDO, 1564АП3У2, 1594ТЛ2Т)
Power: TPS62161/2/3 replaced by a two-stage "DC/DC + LDO" scheme:
- D5 1393ЕУ014 +15 V -> +5,02 V (maker's spec v2.1 pinout; FB 40,2k/10k,
  CL 909 Ohm, soft start 100k/0,22u, EXT compensation 10k + 0,1u,
  L8 56 uH, VD2 2Д2990А, 22 uF + 100 uF tantalum output); PG -> MCU reset
- D6 1158ЕН3.3ВХ +5 V -> +3,3 V, D7 1325ЕН1.8У +5 V -> +1,8 V with a
  +5V copper heat spreader on F.Cu/B.Cu (up to 1,3 W)
- 1272ПН3Т is not used (customer decision)

SPI level shifting: SN74LVC125A -> 1564АП3У2 from +3,3 V with 1 kOhm series
resistors on all five 5 V inputs including 1OE#; SN74AHCT1G125 -> two
inverters of 1594ТЛ2Т from +5 V.

Connectivity changes in tools/eco.py; verified against the intended rev E
netlist and, for untouched parts, against rev C. ERC 0; board re-placed and
routed, DRC with schematic parity 0. Land patterns of all new domestic parts
are PLACEHOLDERS (not for fabrication). tools/pro_merge.py restores the
schematic settings that pcbnew drops from the .kicad_pro.

Co-Authored-By: Claude Opus 5.5 <noreply@anthropic.com>
Claude-Session: https://claude.ai/code/session_018GorfTmWz53k1K9rRxWMAW
Parts:
- removed C52: 10u, Capacitor_SMD:C_1206_3216Metric, symbol DDS:C
- removed C53: 100n, Capacitor_SMD:C_0603_1608Metric, symbol DDS:C
- removed L10, L9: 2.2u, Inductor_SMD:L_Changjiang_FNR4020S, symbol DDS:L
- added C47: 10u, Capacitor_SMD:C_1206_3216Metric, symbol DDS:C
- added C53: 100u, Capacitor_Tantalum_SMD:CP_EIA-7343-31_Kemet-D, symbol DDS:C_Pol
- added C55, C56: 1u, Capacitor_SMD:C_0603_1608Metric, symbol DDS:C
- added C57, C58: 10u, Capacitor_Tantalum_SMD:CP_EIA-3528-21_Kemet-B, symbol DDS:C_Pol
- added C59, C60: 100n, Capacitor_SMD:C_0603_1608Metric, symbol DDS:C
- added R83: 909R, Resistor_SMD:R_0603_1608Metric, symbol DDS:R
- added R84: 100k, Resistor_SMD:R_0603_1608Metric, symbol DDS:R
- added R85, R87: 10k, Resistor_SMD:R_0603_1608Metric, symbol DDS:R
- added R86: 40.2k, Resistor_SMD:R_0603_1608Metric, symbol DDS:R
- added VD2: 2Д2990А, DDS:D_SMA_2D2990A_PLACEHOLDER, symbol DDS:VD_Schottky
- C49: value 10u -> 220n; footprint Capacitor_SMD:C_1206_3216Metric -> Capacitor_SMD:C_0603_1608Metric; Напряжение 25V -> 50V
- C51, C54: value 22u -> 100n; footprint Capacitor_SMD:C_1206_3216Metric -> Capacitor_SMD:C_0603_1608Metric; Напряжение 10V -> 50V
- D5: value TPS62163DSGR -> 1393ЕУ014; footprint Package_SON:Texas_DSG0008A_WSON-8-1EP_2x2mm_P0.5mm_EP0.9x1.6mm -> DDS:4112.16-15.01_1393EU014_PLACEHOLDER; symbol DDS:TPS6216x -> DDS:1393EU014; Примечание +5 В -> DC/DC +15 -> +5 В; корпус 4112.16-15.01 — посадочное место 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
- D6: value TPS62162DSGR -> 1158ЕН3.3ВХ; footprint Package_SON:Texas_DSG0008A_WSON-8-1EP_2x2mm_P0.5mm_EP0.9x1.6mm -> DDS:KT-93-1_PLACEHOLDER; symbol DDS:TPS6216x -> DDS:LDO_1158; Примечание +3,3 В -> LDO +3,3 В
- D7: value TPS62161DSGR -> 1325ЕН1.8У; footprint Package_SON:Texas_DSG0008A_WSON-8-1EP_2x2mm_P0.5mm_EP0.9x1.6mm -> DDS:KT-93-1_PLACEHOLDER; symbol DDS:TPS6216x -> DDS:LDO_1325; Примечание +1,8 В -> LDO +1,8 В
- L8: value 2.2u -> 56u; footprint Inductor_SMD:L_Changjiang_FNR4020S -> DDS:L_10.4x10.4_ID1_PLACEHOLDER; Примечание Isat >= 1,5 А -> ИД1-56, Iнас >= 1,6 А (посадочное место — уточнить по ТУ)
- R88: renamed from R78; Примечание (none) -> признак +3,3 В для МК
- renumbered C47 to C48, C48 to C52
Connections:
- net +1V8: now also D7.1 (OUT), C58.1, C60.1; no longer C54.1, D7.6 (VOS)
- net +3V3: now also D6.3 (OUT), R88.1, C57.1, C59.1; no longer C51.1, D6.6 (VOS)
- net +5V: now also C54.1, D6.1 (IN), C53.1, C55.1, C56.1, R86.1; no longer C49.1, C50.1, D5.6 (VOS), D6.2 (VIN), D6.3 (EN), D7.3 (EN), R88.1
- net DDS_PGOOD: no longer D6.8 (PG), D7.8 (PG)
- net GND: now also D5.11 (GND2), D5.12 (GND3), D6.2 (GND), D7.3 (GND), C47.2, C53.2, C55.2, C56.2, C57.2, C58.2, C59.2, C60.2, R87.2, VD2.2 (A); no longer C51.2, D5.1 (PGND), D5.4 (AGND), D5.9 (EP), D6.1 (PGND), D6.4 (AGND), D6.5 (FB), D6.9 (EP), D7.1 (PGND), D7.4 (AGND), D7.5 (FB), D7.9 (EP)
- net MCU_RESETn: now also D5.13 (PG); no longer D5.8 (PG)
- net VIN_PROT: now also D5.1 (VIN1), C47.1, R83.1, R84.1
- net at L8.1: now also C51.2, D5.14 (SW1), D5.15 (SW2), VD2.1 (K); no longer D5.7 (SW)
- new net: D5.6 (CL), R83.2
- new net: D5.8 (EXT), R85.1
- new net: C50.1, R85.2
- new net: C51.1, D5.4 (BST)
- new net: C49.1, D5.9 (SS), R84.2
- new net: D5.10 (FB), R86.2, R87.1
- no-connect marks 0 -> 2
Other:
- note added: "1. Вход +15 В ±5 %; допустимое входное напряжение D5 9–20 В (порог UVLO 8,0/8,5 В)."
- note added: "3. Ёмкости керамических конденсаторов указаны эффективными при рабочем напряжении, X7R."
- note added: "4. Контур VIN–SW–VD2–GND и C46, C47, C48 — минимальной площади у выводов D5."
- note added: "5. Бюджет +5 В: D7 до 0,4 А, D6 до 0,15 А, МК и логика до 0,06 А — итого до 0,65 А."
- note added: "6. Рассеяние: D7 до 1,3 Вт ((5 − 1,8) В · 0,4 А), D6 до 0,26 Вт; D5 с диодом ≈ 0,4 Вт."
- note added: "7. Корпуса D5–D7, VD2, L8 — посадочные места предварительные, уточнить по ТУ."
- note added: "LDO +1,8 В: CVDD/DVDD DDS"
- note added: "LDO +3,3 В: AVDD/PVDD DDS, генератор, буфер SPI"
- note added: "PG D5 — сброс МК до появления +5 В; вывод ON D5 не подключён (включено)"
- note added: "R88: признак наличия +3,3 В для МК (вход DDS_PGOOD)"
- note added: "U = 1,0 В·(1 + R86/R87) = 5,02 В; порог тока ≈ R83·0,5 мА/R(ключа) ≈ 1,6 А;"
- note added: "плавный пуск ≈ 1,5 мс (R84, C49); коррекция «универсальная» (R85, C50)"
- note removed: "1. Вход +15 В ±5 %; напряжение на входе D5 должно оставаться ниже 17 В."
- note removed: "3. Ёмкости указаны эффективными при рабочем напряжении, диэлектрик X7R."
- note removed: "4. Тепловые площадки D5–D7 соединить с GND; контуры SW — минимальной длины."
- note removed: "5. PG D5 формирует сброс МК; PG D6, D7 — признак готовности питания DDS."
- note removed: "6. Бюджет: 1,8 В <= 0,4 А (DDS); 3,3 В <= 0,2 А + генератор G1 (уточнить)."
- note removed: "PG D6, D7 — монтажное И: питание DDS в норме"
- moved on the sheet: C46, C48, C52, L8, R88
