File: DDS_47_51.kicad_pcb (KiCad board)
At the start: 4 copper layers, 120 x 50 mm, 160 parts, among them X1 PLD-6, X2 PLS-2

Commit message: Rev E: domestic regulators and logic (1393ЕУ014 + LDO, 1564АП3У2, 1594ТЛ2Т)
Power: TPS62161/2/3 replaced by a two-stage "DC/DC + LDO" scheme:
- D5 1393ЕУ014 +15 V -> +5,02 V (maker's spec v2.1 pinout; FB 40,2k/10k,
  CL 909 Ohm, soft start 100k/0,22u, EXT compensation 10k + 0,1u,
  L8 56 uH, VD2 2Д2990А, 22 uF + 100 uF tantalum output); PG -> MCU reset
- D6 1158ЕН3.3ВХ +5 V -> +3,3 V, D7 1325ЕН1.8У +5 V -> +1,8 V with a
  +5V copper heat spreader on F.Cu/B.Cu (up to 1,3 W)
- 1272ПН3Т is not used (customer decision)

SPI level shifting: SN74LVC125A -> 1564АП3У2 from +3,3 V with 1 kOhm series
resistors on all five 5 V inputs including 1OE#; SN74AHCT1G125 -> two
inverters of 1594ТЛ2Т from +5 V.

Connectivity changes in tools/eco.py; verified against the intended rev E
netlist and, for untouched parts, against rev C. ERC 0; board re-placed and
routed, DRC with schematic parity 0. Land patterns of all new domestic parts
are PLACEHOLDERS (not for fabrication). tools/pro_merge.py restores the
schematic settings that pcbnew drops from the .kicad_pro.

Co-Authored-By: Claude Opus 5.5 <noreply@anthropic.com>
Claude-Session: https://claude.ai/code/session_018GorfTmWz53k1K9rRxWMAW
Parts:
- removed L10, L9: 2.2u, Inductor_SMD:L_Changjiang_FNR4020S
- added C55: 1u, Capacitor_SMD:C_0603_1608Metric, F.Cu at (120.4, 135.0)
- added C56: 1u, Capacitor_SMD:C_0603_1608Metric, F.Cu at (132.8, 135.0)
- added C57: 10u, Capacitor_Tantalum_SMD:CP_EIA-3528-21_Kemet-B, F.Cu at (123.0, 135.0)
- added C58: 10u, Capacitor_Tantalum_SMD:CP_EIA-3528-21_Kemet-B, F.Cu at (128.4, 135.0)
- added C59: 100n, Capacitor_SMD:C_0603_1608Metric, F.Cu at (125.6, 135.0)
- added C60: 100n, Capacitor_SMD:C_0603_1608Metric, F.Cu at (131.0, 135.0)
- added R79: 10k, Resistor_SMD:R_0603_1608Metric, F.Cu at (174.4, 105.6)
- added R80: 10k, Resistor_SMD:R_0603_1608Metric, F.Cu at (174.4, 107.3)
- added R81: 1k, Resistor_SMD:R_0603_1608Metric, F.Cu at (168.5, 126.6)
- added R82: 100k, Resistor_SMD:R_0603_1608Metric, F.Cu at (168.5, 128.4)
- added R83: 909R, Resistor_SMD:R_0603_1608Metric, F.Cu at (114.4, 137.6)
- added R84: 100k, Resistor_SMD:R_0603_1608Metric, F.Cu at (124.0, 114.8)
- added R85: 10k, Resistor_SMD:R_0603_1608Metric, F.Cu at (118.0, 137.6)
- added R86: 40.2k, Resistor_SMD:R_0603_1608Metric, F.Cu at (120.4, 114.8)
- added R87: 10k, Resistor_SMD:R_0603_1608Metric, F.Cu at (122.2, 114.8)
- added R88: 47k, Resistor_SMD:R_0603_1608Metric, F.Cu at (122.0, 104.0)
- added VD2: 2Д2990А, DDS:D_SMA_2D2990A_PLACEHOLDER, F.Cu at (102.6, 118.0)
- C47: value 100n -> 10u; footprint Capacitor_SMD:C_0603_1608Metric -> Capacitor_SMD:C_1206_3216Metric
- C48, C51, C54: value 22u -> 100n; footprint Capacitor_SMD:C_1206_3216Metric -> Capacitor_SMD:C_0603_1608Metric
- C49: value 10u -> 220n; footprint Capacitor_SMD:C_1206_3216Metric -> Capacitor_SMD:C_0603_1608Metric
- C52: value 10u -> 22u
- C53: value 100n -> 100u; footprint Capacitor_SMD:C_0603_1608Metric -> Capacitor_Tantalum_SMD:CP_EIA-7343-31_Kemet-D
- D3: value SN74LVC125APWR -> 1564АП3У2; footprint Package_SO:TSSOP-14_4.4x5mm_P0.65mm -> DDS:SOIC-20W_1564AP3U2_PLACEHOLDER
- D4: value SN74AHCT1G125DBVR -> 1594ТЛ2Т; footprint Package_TO_SOT_SMD:SOT-23-5 -> DDS:SOIC-14_1594TL2T_PLACEHOLDER
- D5: value TPS62163DSGR -> 1393ЕУ014; footprint Package_SON:Texas_DSG0008A_WSON-8-1EP_2x2mm_P0.5mm_EP0.9x1.6mm -> DDS:4112.16-15.01_1393EU014_PLACEHOLDER
- D6: value TPS62162DSGR -> 1158ЕН3.3ВХ; footprint Package_SON:Texas_DSG0008A_WSON-8-1EP_2x2mm_P0.5mm_EP0.9x1.6mm -> DDS:KT-93-1_PLACEHOLDER
- D7: value TPS62161DSGR -> 1325ЕН1.8У; footprint Package_SON:Texas_DSG0008A_WSON-8-1EP_2x2mm_P0.5mm_EP0.9x1.6mm -> DDS:KT-93-1_PLACEHOLDER
- L8: value 2.2u -> 56u; footprint Inductor_SMD:L_Changjiang_FNR4020S -> DDS:L_10.4x10.4_ID1_PLACEHOLDER
- R65, R66: value 10k -> 1k
- R68, R70, R71: value 33R -> 1k
- R69: value 33R -> 10k
- R73, R74, R75: value 10k -> 33R
- R76: value 1k -> 33R
- R77: value 100k -> 10k
- R78: value 47k -> 10k
- moved R78 48.7 mm to (174.4, 103.9), turned to 0 degrees
- moved L8 33.0 mm to (107.2, 107.0)
- moved R77 24.5 mm to (174.4, 102.2)
- moved D7 21.8 mm to (130.3, 126.0), turned to 90 degrees
- moved R76 20.5 mm to (170.4, 103.6), turned to 90 degrees
- moved C51 19.3 mm to (116.2, 137.6)
- moved C45 16.5 mm to (174.0, 133.6)
- moved R67 16.1 mm to (161.6, 123.6), turned to 90 degrees
- moved R63 15.9 mm to (166.6, 123.6), turned to 90 degrees
- moved C50 15.8 mm to (118.0, 141.0), turned to 90 degrees
- moved C48 15.1 mm to (112.6, 137.6)
- moved R72 14.4 mm to (169.2, 123.6), turned to 90 degrees
- moved C49 14.3 mm to (125.8, 114.8)
- moved R73 13.8 mm to (162.8, 103.6), turned to 90 degrees
- moved R69 13.7 mm to (164.1, 123.6), turned to 90 degrees
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Connections:
- C48 pad 1: +5V -> /Питание/VIN_PROT
- C49 pad 1: +5V -> Net-(D5-SS)
- C50 pad 1: +5V -> Net-(C50-Pad1)
- C51 pad 1: +3V3 -> Net-(D5-BST)
- C51 pad 2: GND -> Net-(D5-SW1)
- C54 pad 1: +1V8 -> +5V
- D3 pad 1: /Контроллер/BUF_OEn -> Net-(D3.1-EN)
- D3 pad 10: /Контроллер/BUF_OEn -> GND
- D3 pad 11: /Контроллер/RST_BUF -> GND
- D3 pad 12: /Контроллер/MCU_DDS_RESET -> /Контроллер/RST_BUF
- D3 pad 13: /Контроллер/BUF_OEn -> GND
- D3 pad 14: +3V3 -> /Контроллер/CS_BUF
- D3 pad 2: /Контроллер/MCU_SCK -> Net-(D3-Pad2)
- D3 pad 3: /Контроллер/SCK_BUF -> unconnected-(D3-Pad3)
- D3 pad 4: /Контроллер/BUF_OEn -> Net-(D3-Pad4)
- D3 pad 5: /Контроллер/MCU_MOSI -> unconnected-(D3-Pad5)
- D3 pad 6: /Контроллер/MOSI_BUF -> Net-(D3-Pad6)
- D3 pad 7: GND -> unconnected-(D3-Pad7)
- D3 pad 8: /Контроллер/CS_BUF -> Net-(D3-Pad8)
- D3 pad 9: /Контроллер/MCU_CS -> unconnected-(D3-Pad9)
- D4 pad 1: GND -> /Контроллер/SDO_BUF
- D4 pad 2: /Контроллер/SDO_BUF -> /Контроллер/SDO_INV
- D4 pad 3: GND -> /Контроллер/SDO_INV
- D4 pad 5: +5V -> GND
- D5 pad 1: GND -> /Питание/VIN_PROT
- D5 pad 4: GND -> Net-(D5-BST)
- D5 pad 6: +5V -> Net-(D5-CL)
- D5 pad 7: Net-(D5-SW) -> unconnected-(D5-ON-Pad7)
- D5 pad 8: MCU_RESETn -> Net-(D5-EXT)
- D5 pad 9: GND -> Net-(D5-SS)
- D6 pad 1: GND -> +5V
- D6 pad 2: +5V -> GND
- D6 pad 3: +5V -> +3V3
- D7 pad 1: GND -> +1V8
- D7 pad 3: +5V -> GND
- L8 pad 1: Net-(D5-SW) -> Net-(D5-SW1)
- R63 pad 1: /Контроллер/MCU_SCK -> +5V
- R63 pad 2: GND -> /Контроллер/MCU_CS
- R64 pad 1: /Контроллер/MCU_MOSI -> +3V3
- R64 pad 2: GND -> /Контроллер/BUF_OEn
- R65 pad 1: +5V -> /Контроллер/BUF_OEn
- R65 pad 2: /Контроллер/MCU_CS -> Net-(D3.1-EN)
- R66 pad 1: /Контроллер/MCU_DDS_RESET -> /Контроллер/MCU_SCK
- R66 pad 2: GND -> Net-(D3-Pad2)
- R67 pad 1: +3V3 -> /Контроллер/MCU_SCK
- R67 pad 2: /Контроллер/BUF_OEn -> GND
- R68 pad 1: /Контроллер/SCK_BUF -> /Контроллер/MCU_MOSI
- R68 pad 2: DDS_SCK -> Net-(D3-Pad4)
- R69 pad 1: /Контроллер/MOSI_BUF -> /Контроллер/MCU_MOSI
- R69 pad 2: DDS_SDI -> GND
- R70 pad 1: /Контроллер/CS_BUF -> /Контроллер/MCU_CS
- R70 pad 2: DDS_SCSn -> Net-(D3-Pad6)
- R71 pad 1: /Контроллер/RST_BUF -> /Контроллер/MCU_DDS_RESET
- R71 pad 2: DDS_RSTn -> Net-(D3-Pad8)
- R72 pad 1: DDS_SCK -> /Контроллер/MCU_DDS_RESET
- R73 pad 1: DDS_SDI -> /Контроллер/SCK_BUF
- R73 pad 2: GND -> DDS_SCK
- R74 pad 1: +3V3 -> /Контроллер/MOSI_BUF
- R74 pad 2: DDS_SCSn -> DDS_SDI
- R75 pad 1: DDS_RSTn -> /Контроллер/CS_BUF
- R75 pad 2: GND -> DDS_SCSn
- R76 pad 1: DDS_SDO -> /Контроллер/RST_BUF
- R76 pad 2: /Контроллер/SDO_BUF -> DDS_RSTn
- R77 pad 1: /Контроллер/SDO_BUF -> DDS_SCK
- R78 pad 1: +5V -> DDS_SDI
- R78 pad 2: DDS_PGOOD -> GND
Routing:
- net +3V3: track 201.4 -> 259.2 mm, vias 6 -> 5
- net Net-(D5-SW1): track 0.00 -> 43.3 mm, vias 0 -> 2
- net GND: track 262.3 -> 300.7 mm, vias 320 -> 283
- net /Питание/VIN_PROT: track 12.6 -> 46.5 mm
- net /Контроллер/BUF_OEn: track 50.9 -> 25.8 mm
- net /Контроллер/APPLYn: track 39.7 -> 60.2 mm, vias 2 -> 1
- net Net-(D5-SS): track 0.00 -> 18.2 mm, vias 0 -> 2
- net DDS_SCK: track 21.5 -> 36.4 mm, vias 0 -> 3
- net DDS_SDI: track 23.3 -> 37.8 mm
- net +3V3_A: track 107.9 -> 94.3 mm, vias 3 -> 4
- net /Контроллер/DIP6: track 34.3 -> 47.6 mm
- net /Контроллер/DIP9: track 32.0 -> 43.8 mm, vias 1 -> 3
- net Net-(D5-FB): track 0.00 -> 10.7 mm, vias 0 -> 2
- net +1V8: track 156.3 -> 145.8 mm, vias 2 -> 4
- net DDS_SCSn: track 21.2 -> 31.8 mm, vias 0 -> 4
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- added copper zone on B.Cu, net +5V
- added copper zone on F.Cu, net +5V
