File: DDS_47_51.kicad_sch (KiCad schematic)
At the start: 0 parts

Commit message: Switch to rev C: three-sheet schematic in project root
Replace the 10-sheet rev B schematic (index + 9 sheets) with the rev C
layout: DDS (A2), controller (A2) and power (A3), with no index sheet.
Connectivity is unchanged: a fresh KiCad 10.0.6 netlist comparison of
rev B and rev C gives 170 components and 139 nets with identical pin sets.

Reorganise the folder: KiCad sources and READMEs stay in the root;
design notes in docs/, PDF/BOM/netlist exports in output/, ERC report in
reports/, connectivity reference in verification/, scripts in tools/
(rev B/C generators kept in tools/legacy/). Add tools/netcompare.py.

ERC is still not clean (849 violations: 671 off-grid, 170 symbol library,
8 power pins not driven). Not a manufacturing release.

Co-Authored-By: Claude Opus 5.5 <noreply@anthropic.com>
Claude-Session: https://claude.ai/code/session_018GorfTmWz53k1K9rRxWMAW
Parts:
- added C10, C11, C12, C35, C36, C37, C38: 10u / 10V, symbol Local:C
- added C13: 100n / U1.1, symbol Local:C
- added C14: 100n / U1.9, symbol Local:C
- added C15: 100n / U1.14, symbol Local:C
- added C16: 100n / U1.15, symbol Local:C
- added C17: 100n / U1.16, symbol Local:C
- added C18: 100n / U1.21, symbol Local:C
- added C19: 100n / U1.26, symbol Local:C
- added C20: 100n / U1.27, symbol Local:C
- added C21: 100n / U1.30, symbol Local:C
- added C22: 100n / U1.31, symbol Local:C
- added C23: 100n / U1.36, symbol Local:C
- added C24: 100n / U1.39, symbol Local:C
- added C25: 100n / U1.40, symbol Local:C
- added C26: 100n / U1.45, symbol Local:C
- added C27: 100n / U1.47, symbol Local:C
- added C28: 100n / U1.51, symbol Local:C
- added C29: 100n / U1.60, symbol Local:C
- added C30: 100n / U1.61, symbol Local:C
- added C31: 100n / U1.69, symbol Local:C
- added C32: 100n / U1.75, symbol Local:C
- added C33: 100n / U1.82, symbol Local:C
- added C34: 100n / U1.94, symbol Local:C
- added C47: 100n, symbol Local:C
- added C48: 1u, symbol Local:C
- added C49, C50, C51: 10n C0G, symbol Local:C
- added C52, C54: 56p C0G, symbol Local:C
- added C53: 91p C0G, symbol Local:C
- added FB1, FB2, FB3: 600R@100MHz / 1A, symbol Local:L
- added G1: GK361-TK-02 / DNP, symbol Local:GK361_UNVERIFIED
- added J2: SMA EXT / 480MHz, symbol Local:J2
- added J3: SMA OUT / 50 ohm, symbol Local:J2
- added L4, L7: 51nH, symbol Local:L
- added L5, L6: 200nH, symbol Local:L
- added R10, R11, R12, R13, R14, R15, R16, R17, R18, R19, R20, R21, R22, R23, R24, R25, R26, R27, R28, R29, R30, R31, R32, R33, R34, R35, R7, R8, R9: 100k, symbol Local:R
- added R2, R3: 7.15k / 0.1%, symbol Local:R
- added R4, R5, R6, R71: 10k, symbol Local:R
- added R66: 10k / DNP, symbol Local:R
- added R67, R68: 0R / DNP, symbol Local:R
- added R69: 100R / 1%, symbol Local:R
- added R70: 49.9R / 1%, symbol Local:R
- added R72, R73, R74, R75: 49.9R / 0.1%, symbol Local:R
- added R76: 5.76R 1%, symbol Local:R
- added R77, R78: 866R 1%, symbol Local:R
- added SW14: CSEL / closed=EXT, symbol Local:SW_SPST
- added U1: 1508PL8T, symbol Local:1508PL8T
Connections:
- new net: C53.1, L5.2, L6.1
- new net: C54.1, L6.2, L7.1
- new net: C51.2, L4.1
- new net: C52.1, L4.2, L5.1
- new net: L7.2, R76.1, R77.1
- new net +1V8: C13.1, C15.1, C16.1, C29.1, C30.1, C32.1, C33.1, C35.1, FB3.1, U1.1 (CVDD), U1.14 (CVDD), U1.15 (CVDD), U1.60 (CVDD), U1.61 (CVDD), U1.75 (CVDD), U1.82 (CVDD)
- new net +1V8_Q: C12.1, C17.1, C23.1, C26.1, C27.1, C38.1, FB3.2, U1.16 (DVDD), U1.36 (DVDD2), U1.45 (DVDD1), U1.47 (DVDD)
- new net +3V3: C14.1, C31.1, C34.1, C36.1, FB1.1, FB2.1, R4.1, R5.1, R6.1, SW14.1 (A), U1.69 (PVDD), U1.9 (PVDD), U1.94 (PVDD)
- new net +3V3_A: C10.1, C18.1, C19.1, C20.1, C21.1, C22.1, C24.1, C25.1, C28.1, C37.1, FB1.2, U1.21 (AVDD), U1.26 (AVDD), U1.27 (AVDD), U1.30 (AVDD2), U1.31 (AVDD2), U1.39 (AVDD1), U1.40 (AVDD1), U1.51 (CMP_VDD)
- new net +3V3_OSC: C11.1, C47.1, C48.1, FB2.2, G1.6 (VCC?), R66.1
- new net ADR: R7.1, U1.11 (ADR)
- new net CLKDM: C50.1, U1.19 (CLKDM)
- new net CLKDP: C49.2, U1.18 (CLKDP)
- new net CLKM: R68.2, R69.2, U1.23 (CLKM)
- new net CLKP: R67.2, R69.1, U1.24 (CLKP)
- new net CSEL: R71.1, SW14.2 (B), U1.13 (CSEL)
- new net CSn: R4.2, U1.8 (CSn)
- new net DATA_0: R20.1, U1.78 (DATA_0)
- new net DATA_1: R21.1, U1.79 (DATA_1)
- new net DATA_10: R30.1, U1.92 (DATA_10)
- new net DATA_11: R31.1, U1.93 (DATA_11)
- new net DATA_12: R32.1, U1.95 (DATA_12)
- new net DATA_13: R33.1, U1.96 (DATA_13)
- new net DATA_14: R34.1, U1.97 (DATA_14)
- new net DATA_15: R35.1, U1.98 (DATA_15)
- new net DATA_2: R22.1, U1.80 (DATA_2)
- new net DATA_3: R23.1, U1.81 (DATA_3)
- new net DATA_4: R24.1, U1.83 (DATA_4)
- new net DATA_5: R25.1, U1.84 (DATA_5)
- new net DATA_6: R26.1, U1.87 (DATA_6)
- new net DATA_7: R27.1, U1.88 (DATA_7)
- new net DATA_8: R28.1, U1.89 (DATA_8)
- new net DATA_9: R29.1, U1.90 (DATA_9)
- new net DDS_RSTn: U1.10 (RSTn)
- new net DDS_SCK: U1.2 (SCK)
- new net DDS_SCSn: U1.6 (SCSn)
- new net DDS_SDI: U1.3 (SDI)
- new net DDS_SDO: U1.5 (SDO)
- new net EXT_CLK: C49.1, J2.1, R70.1
- new net GND: C10.2, C11.2, C12.2, C13.2, C14.2, C15.2, C16.2, C17.2, C18.2, C19.2, C20.2, C21.2, C22.2, C23.2, C24.2, C25.2, C26.2, C27.2, C28.2, C29.2, C30.2, C31.2, C32.2, C33.2, C34.2, C35.2, C36.2, C37.2, C38.2, C47.2, C48.2, C50.2, C52.2, C53.2, C54.2, G1.3 (GND?), J2.2, J3.2, R10.2, R11.2, R12.2, R13.2, R14.2, R15.2, R16.2, R17.2, R18.2, R19.2, R2.2, R20.2, R21.2, R22.2, R23.2, R24.2, R25.2, R26.2, R27.2, R28.2, R29.2, R3.2, R30.2, R31.2, R32.2, R33.2, R34.2, R35.2, R7.2, R70.2, R71.2, R72.2, R73.2, R74.2, R75.2, R77.2, R78.2, R8.2, R9.2, U1.12 (PGND), U1.17 (AGND), U1.20 (AGND), U1.22 (AGND), U1.25 (AGND), U1.29 (AGND), U1.32 (AGND), U1.35 (AGND), U1.38 (AGND), U1.4 (CGND), U1.41 (AGND), U1.44 (AGND), U1.46 (AGND), U1.48 (CMP_GND), U1.49 (CMP_INM), U1.50 (CMP_INP), U1.54 (CMP_GND), U1.55 (CGND), U1.64 (CGND), U1.65 (CGND), U1.66 (PGND), U1.72 (CGND), U1.85 (CGND), U1.86 (CGND), U1.91 (PGND), U1.99 (CGND)
- new net IREF1: R2.1, U1.37 (IREF1)
- new net IREF2: R3.1, U1.28 (IREF2)
- new net OSC_EN: G1.1 (EN?), R66.2
- new net OSC_M: G1.5 (OUT_N?), R68.1
- new net OSC_P: G1.4 (OUT_P?), R67.1
- new net OUTM1: R73.1, U1.42 (OUTM1)
- new net OUTM2: R75.1, U1.33 (OUTM2)
- new net OUTP1: C51.1, R72.1, U1.43 (OUTP1)
- new net OUTP2: R74.1, U1.34 (OUTP2)
- new net RDn: R5.2, U1.76 (RDn)
- new net RF_OUT: J3.1, R76.2, R78.1
- new net SEL1_0: R14.1, U1.67 (SEL1_0)
- new net SEL1_1: R15.1, U1.68 (SEL1_1)
- new net SEL1_2: R16.1, U1.70 (SEL1_2)
- new net SEL1_3: R17.1, U1.71 (SEL1_3)
- new net SEL1_4: R18.1, U1.73 (SEL1_4)
- new net SEL1_5: R19.1, U1.74 (SEL1_5)
- new net SEL2_0: R8.1, U1.56 (SEL2_0)
- new net SEL2_1: R9.1, U1.57 (SEL2_1)
- new net SEL2_2: R10.1, U1.58 (SEL2_2)
- new net SEL2_3: R11.1, U1.59 (SEL2_3)
- new net SEL2_4: R12.1, U1.62 (SEL2_4)
- new net SEL2_5: R13.1, U1.63 (SEL2_5)
- new net WRn: R6.2, U1.77 (WRn)
- no-connect marks 0 -> 5
Other:
- removed sheet 01_power
- removed sheet 02_dds
- removed sheet 03_bias
- removed sheet 04_bypass
- removed sheet 05_mcu
- removed sheet 06_ui
- removed sheet 07_spi
- removed sheet 08_clock
- removed sheet 09_rf
- added sheet Controller (02_controller.kicad_sch)
- added sheet Power supply / +15 V input (03_power.kicad_sch)
- note added: "01 DDS / 47-51 MHz / 1 kHz / -10 dBm"
- note added: "480 MHz clock / G1 unverified, DNP"
- note added: "Local bypass: place at the indicated U1 pins"
- note added: "RF: DAC loads / 7-pole LPF / pi attenuator"
- note added: "Unused input pull-downs"
- note removed: "DDS 47-51 MHz | 1 kHz step | -10 dBm into 50 ohm 1508PL8T + 1887VE7T | +15 V | target PCB <=80 x 50 mm"
- note removed: "REVISION B - ENGINEERING DRAFT All circuit sections connected. G1 blocked pending manufacturer passport. PCB placement, thermal/noise validation and output calibration remain open. Matching global labels connect electrically across all sheets."
- note removed: "Read README_RU.md for assembly choices, firmware contract, sources and validation limits. Open DDS_47_51.kicad_pro. PDF and netlist come from this same schematic."
- title: DDS 47-51 MHz / revision B / circuit draft -> DDS, clock and RF output

Commit message: Rev D schematic: ГОСТ symbols and designators in KiCad, footprints
- Three sheets regenerated by tools/dds_build.py (DDS A2, controller A3,
  power A2) with ГОСТ 2.743 symbols, ГОСТ 2.710 designators (D1.1, XW1, S2)
  and a ГОСТ 2.104 drawing sheet (lib/GOST_E3.kicad_wks).
- Connectivity identical to rev C (tools/netcompare.py with
  verification/refmap_revC_to_revD.json): 160 components, 139 nets; the 12
  single DIP switches are grouped into DIP-8 + DIP-4 packages.
- ERC: 0 errors, 0 warnings. Footprints assigned; project library lib/
  (1508PL8T LQFP-100, 1887VE7T CQFP-64 4203.64-2 preliminary, GK361-TK-02
  placeholder - not confirmed, DNP).
- Old rev C PDF replaced by output/pdf/DDS_47_51_sch.pdf.

Co-Authored-By: Claude Opus 5.5 <noreply@anthropic.com>
Claude-Session: https://claude.ai/code/session_018GorfTmWz53k1K9rRxWMAW
Parts:
- removed C10, C11, C12, C35, C36, C37, C38: 10u / 10V, symbol Local:C
- removed C13: 100n / U1.1, symbol Local:C
- removed C14: 100n / U1.9, symbol Local:C
- removed C15: 100n / U1.14, symbol Local:C
- removed C16: 100n / U1.15, symbol Local:C
- removed C17: 100n / U1.16, symbol Local:C
- removed C18: 100n / U1.21, symbol Local:C
- removed C19: 100n / U1.26, symbol Local:C
- removed C20: 100n / U1.27, symbol Local:C
- removed C21: 100n / U1.30, symbol Local:C
- removed C22: 100n / U1.31, symbol Local:C
- removed C23: 100n / U1.36, symbol Local:C
- removed C24: 100n / U1.39, symbol Local:C
- removed C25: 100n / U1.40, symbol Local:C
- removed C26: 100n / U1.45, symbol Local:C
- removed C27: 100n / U1.47, symbol Local:C
- removed C28: 100n / U1.51, symbol Local:C
- removed C29: 100n / U1.60, symbol Local:C
- removed C30: 100n / U1.61, symbol Local:C
- removed C31: 100n / U1.69, symbol Local:C
- removed C32: 100n / U1.75, symbol Local:C
- removed C33: 100n / U1.82, symbol Local:C
- removed C34: 100n / U1.94, symbol Local:C
- removed C47: 100n, symbol Local:C
- removed C48: 1u, symbol Local:C
- removed C49, C50, C51: 10n C0G, symbol Local:C
- removed C52, C54: 56p C0G, symbol Local:C
- removed C53: 91p C0G, symbol Local:C
- removed FB1, FB2, FB3: 600R@100MHz / 1A, symbol Local:L
- removed G1: GK361-TK-02 / DNP, symbol Local:GK361_UNVERIFIED
- removed J2: SMA EXT / 480MHz, symbol Local:J2
- removed J3: SMA OUT / 50 ohm, symbol Local:J2
- removed L4, L7: 51nH, symbol Local:L
- removed L5, L6: 200nH, symbol Local:L
- removed R10, R11, R12, R13, R14, R15, R16, R17, R18, R19, R20, R21, R22, R23, R24, R25, R26, R27, R28, R29, R30, R31, R32, R33, R34, R35, R7, R8, R9: 100k, symbol Local:R
- removed R2, R3: 7.15k / 0.1%, symbol Local:R
- removed R4, R5, R6, R71: 10k, symbol Local:R
- removed R66: 10k / DNP, symbol Local:R
- removed R67, R68: 0R / DNP, symbol Local:R
- removed R69: 100R / 1%, symbol Local:R
- removed R70: 49.9R / 1%, symbol Local:R
- removed R72, R73, R74, R75: 49.9R / 0.1%, symbol Local:R
- removed R76: 5.76R 1%, symbol Local:R
- removed R77, R78: 866R 1%, symbol Local:R
- removed SW14: CSEL / closed=EXT, symbol Local:SW_SPST
- removed U1: 1508PL8T, symbol Local:1508PL8T
- added C1: 1u, Capacitor_SMD:C_0603_1608Metric, symbol DDS:C
- added C10, C19, C24, C28, C37, C8, C9: 10u, Capacitor_SMD:C_0805_2012Metric, symbol DDS:C
- added C11, C6: 56p, Capacitor_SMD:C_0603_1608Metric, symbol DDS:C
- added C12, C13, C14, C15, C16, C17, C18, C2, C20, C21, C22, C23, C25, C26, C27, C29, C30, C31, C32, C33, C34, C35, C36: 100n, Capacitor_SMD:C_0603_1608Metric, symbol DDS:C
- added C3, C4, C5: 10n, Capacitor_SMD:C_0603_1608Metric, symbol DDS:C
- added C7: 91p, Capacitor_SMD:C_0603_1608Metric, symbol DDS:C
- added D1: 1508ПЛ8Т, DDS:LQFP-100_14x14mm_P0.5mm_1508PL8T, symbol DDS:1508PL8T
- added G1: ГК361-ТК-02, DDS:OSC_6pad_5.0x3.2mm_P1.27mm_GK361_UNVERIFIED, symbol DDS:GK361_UNVERIFIED
- added L1, L7: 51n, Inductor_SMD:L_0603_1608Metric, symbol DDS:L
- added L2, L3, L4: 600R@100MHz, Inductor_SMD:L_0603_1608Metric, symbol DDS:L_Fe
- added L5, L6: 200n, Inductor_SMD:L_0603_1608Metric, symbol DDS:L
- added R1, R5, R7, R8, R9: 10k, Resistor_SMD:R_0603_1608Metric, symbol DDS:R
- added R10, R13, R14, R15, R16, R17, R18, R19, R20, R21, R22, R23, R24, R28, R29, R30, R31, R32, R33, R34, R35, R36, R37, R38, R39, R40, R41, R42, R43: 100k, Resistor_SMD:R_0603_1608Metric, symbol DDS:R
- added R11, R12: 7.15k, Resistor_SMD:R_0603_1608Metric, symbol DDS:R
- added R2, R25, R26, R27, R44: 49.9R, Resistor_SMD:R_0603_1608Metric, symbol DDS:R
- added R3, R4: 0R, Resistor_SMD:R_0603_1608Metric, symbol DDS:R
- added R45: 5.76R, Resistor_SMD:R_0603_1608Metric, symbol DDS:R
- added R46, R47: 866R, Resistor_SMD:R_0603_1608Metric, symbol DDS:R
- added R6: 100R, Resistor_SMD:R_0603_1608Metric, symbol DDS:R
- added S1: DIP-1, Button_Switch_THT:SW_DIP_SPSTx01_Slide_9.78x4.72mm_W7.62mm_P2.54mm, symbol DDS:S_DIP_x01
- added XW1, XW2: SMA, Connector_Coaxial:SMA_Samtec_SMA-J-P-H-ST-EM1_EdgeMount, symbol DDS:XW_Coax
Connections:
- net +1V8: now also C12.1, C13.1, C14.1, C15.1, C16.1, C17.1, C18.1, C19.1, D1.1 (CVDD), D1.14 (CVDD), D1.15 (CVDD), D1.60 (CVDD), D1.61 (CVDD), D1.75 (CVDD), D1.82 (CVDD), L4.1
- net +1V8_Q: now also C10.1, C20.1, C21.1, C22.1, C23.1, C24.1, D1.16 (DVDD), D1.36 (DVDD2), D1.45 (DVDD1), D1.47 (DVDD), L4.2
- net +3V3: now also C25.1, C26.1, C27.1, C28.1, D1.69 (PVDD), D1.9 (PVDD), D1.94 (PVDD), L2.1, L3.1, R7.1, R8.1, R9.1, S1.1
- net +3V3_A: now also C29.1, C30.1, C31.1, C32.1, C33.1, C34.1, C35.1, C36.1, C37.1, C8.1, D1.21 (AVDD), D1.26 (AVDD), D1.27 (AVDD), D1.30 (AVDD2), D1.31 (AVDD2), D1.39 (AVDD1), D1.40 (AVDD1), D1.51 (CMP_VDD), L2.2
- net +3V3_OSC: now also C1.1, C2.1, C9.1, G1.6 (VCC?), L3.2, R1.1
- net ADR: now also D1.11 (ADR), R10.1
- net CLKDM: now also C4.1, D1.19 (CLKDM)
- net CLKDP: now also C3.2, D1.18 (CLKDP)
- net CLKM: now also D1.23 (CLKM), R4.2, R6.2
- net CLKP: now also D1.24 (CLKP), R3.2, R6.1
- net CSEL: now also D1.13 (CSEL), R5.1, S1.2
- net CSn: now also D1.8 (CS), R7.2
- net DATA_0: now also D1.78 (D0), R28.1
- net DATA_1: now also D1.79 (D1), R29.1
- net DATA_10: now also D1.92 (D10), R38.1
- net DATA_11: now also D1.93 (D11), R39.1
- net DATA_12: now also D1.95 (D12), R40.1
- net DATA_13: now also D1.96 (D13), R41.1
- net DATA_14: now also D1.97 (D14), R42.1
- net DATA_15: now also D1.98 (D15), R43.1
- net DATA_2: now also D1.80 (D2), R30.1
- net DATA_3: now also D1.81 (D3), R31.1
- net DATA_4: now also D1.83 (D4), R32.1
- net DATA_5: now also D1.84 (D5), R33.1
- net DATA_6: now also D1.87 (D6), R34.1
- net DATA_7: now also D1.88 (D7), R35.1
- net DATA_8: now also D1.89 (D8), R36.1
- net DATA_9: now also D1.90 (D9), R37.1
- net DDS_RSTn: now also D1.10 (RST)
- net DDS_SCK: now also D1.2 (SCK)
- net DDS_SCSn: now also D1.6 (SCS)
- net DDS_SDI: now also D1.3 (SDI)
- net DDS_SDO: now also D1.5 (SDO)
- net GND: now also C1.2, C10.2, C11.2, C12.2, C13.2, C14.2, C15.2, C16.2, C17.2, C18.2, C19.2, C2.2, C20.2, C21.2, C22.2, C23.2, C24.2, C25.2, C26.2, C27.2, C28.2, C29.2, C30.2, C31.2, C32.2, C33.2, C34.2, C35.2, C36.2, C37.2, C4.2, C6.2, C7.2, C8.2, C9.2, D1.12 (PGND), D1.17 (AGND), D1.20 (AGND), D1.22 (AGND), D1.25 (AGND), D1.29 (AGND), D1.32 (AGND), D1.35 (AGND), D1.38 (AGND), D1.4 (CGND), D1.41 (AGND), D1.44 (AGND), D1.46 (AGND), D1.48 (CMP_GND), D1.49 (CMP_INM), D1.50 (CMP_INP), D1.54 (CMP_GND), D1.55 (CGND), D1.64 (CGND), D1.65 (CGND), D1.66 (PGND), D1.72 (CGND), D1.85 (CGND), D1.86 (CGND), D1.91 (PGND), D1.99 (CGND), G1.3 (GND?), R10.2, R11.2, R12.2, R13.2, R14.2, R15.2, R16.2, R17.2, R18.2, R19.2, R2.2, R20.2, R21.2, R22.2, R23.2, R24.2, R25.2, R26.2, R27.2, R28.2, R29.2, R30.2, R31.2, R32.2, R33.2, R34.2, R35.2, R36.2, R37.2, R38.2, R39.2, R40.2, R41.2, R42.2, R43.2, R44.2, R46.2, R47.2, R5.2, XW1.2, XW2.2
- net IREF1: now also D1.37 (IREF1), R11.1
- net IREF2: now also D1.28 (IREF2), R12.1
- net OUTM1: now also D1.42 (OUTM1), R25.1
- net OUTM2: now also D1.33 (OUTM2), R27.1
- net OUTP1: now also C5.1, D1.43 (OUTP1), R44.1
- net OUTP2: now also D1.34 (OUTP2), R26.1
- net RDn: now also D1.76 (RD), R8.2
- net SEL1_0: now also D1.67 (SEL1[0]), R13.1
- net SEL1_1: now also D1.68 (SEL1[1]), R14.1
- net SEL1_2: now also D1.70 (SEL1[2]), R15.1
- net SEL1_3: now also D1.71 (SEL1[3]), R16.1
- net SEL1_4: now also D1.73 (SEL1[4]), R17.1
- net SEL1_5: now also D1.74 (SEL1[5]), R18.1
- net SEL2_0: now also D1.56 (SEL2[0]), R19.1
- net SEL2_1: now also D1.57 (SEL2[1]), R20.1
- net SEL2_2: now also D1.58 (SEL2[2]), R21.1
- net SEL2_3: now also D1.59 (SEL2[3]), R22.1
- net SEL2_4: now also D1.62 (SEL2[4]), R23.1
- net SEL2_5: now also D1.63 (SEL2[5]), R24.1
- net WRn: now also D1.77 (WR), R9.2
- new net: C6.1, L1.2, L5.1
- new net: C7.1, L5.2, L6.1
- new net: R45.2, R47.1, XW2.1
- new net: C3.1, R2.1, XW1.1
- new net: C5.2, L1.1
- new net: C11.1, L6.2, L7.1
- new net: G1.1 (EN?), R1.2
- new net: G1.5 (OUT-?), R4.1
- new net: L7.2, R45.1, R46.1
- new net: G1.4 (OUT+?), R3.1
Other:
- removed sheet Controller
- removed sheet Power supply / +15 V input
- added sheet Контроллер (02_controller.kicad_sch)
- added sheet Питание (03_power.kicad_sch)
- note added: "1. Сплошной общий полигон земли; AGND, PGND, CGND, CMP_GND соединены на нём."
- note added: "2. Ток полной шкалы ЦАП IFS = 72 В / R = 10,07 мА (R11); напряжение на OUTP/OUTM не более ±0,6 В."
- note added: "3. ФНЧ — Баттерворт 7-го порядка, fср ≈ 70 МГц; номиналы округлены до E24."
- note added: "4. Уровень −10 дБм на 50 Ом устанавливается кодом амплитуды DDS при калибровке."
- note added: "5. Индуктивности L1, L5–L7 — ВЧ с высокой добротностью; проверить Q и SRF по моделям."
- note added: "6. Неиспользуемые выводы DATA, SEL — через резисторы на GND, не напрямую."
- note added: "7. Инициализация: ЦАП2 и компаратор выключены, SYNC/LINK выключены, профиль 0."
- note added: "8. Измерения SFDR и шумов не проводились; схема не является выпуском в производство."
- note added: "C12–C18, C20–C23, C25–C27, C29–C36 0,1 мкФ — у выводов D1,"
- note added: "G1, R1, R3, R4 не устанавливаются: параметры и распиновка"
- note added: "R13–R24 100 кОм ±5 %"
- note added: "R25–R27, R44 49,9 Ом ±0,1 %"
- note added: "R28–R43 100 кОм ±5 %"
- note added: "R7–R9 10 кОм; R10 100 кОм; R11, R12 7,15 кОм ±0,1 %"
- note added: "S1 замкнут: такт с XW1 (CLKD); разомкнут: G1 (CLKP/M)"
- note added: "Аттенюатор ≈1 дБ"
- note added: "Вход 480 МГц, 0 дБм / 50 Ом"
- note added: "Выход 47–51 МГц, −10 дБм / 50 Ом"
- note added: "ГК361-ТК-02 не подтверждены паспортом. Перед установкой"
- note added: "Примечания"
- note added: "ФНЧ 7-го порядка, fср ≈ 70 МГц"
- note added: "Фильтры питания DDS"
- note added: "проверить корпус, выходы LVDS, EN, ток; затем разомкнуть S1."
- note added: "указанных в поле «Размещение»; C19, C24, C28, C37 10 мкФ"
- note removed: "01 DDS / 47-51 MHz / 1 kHz / -10 dBm"
- note removed: "480 MHz clock / G1 unverified, DNP"
- note removed: "Local bypass: place at the indicated U1 pins"
- note removed: "RF: DAC loads / 7-pole LPF / pi attenuator"
- note removed: "Unused input pull-downs"
- title: DDS, clock and RF output -> Синтезатор частоты 47–51 МГц
